File: kicad/main.kicad_pcb (KiCad board)
At the start: 4 copper layers, 98.1 x 39.2 mm, 39 parts, among them M1 TP4056_MODULE, M2 BOOST_MODULE, Q1 AO3407, Q2 2N3904, U1 LM431, U2 Arduino_pro_mini

Commit message: docs: clean up schematic and export to pdf and images
Routing:
- net VCC: track 153.8 -> 161.5 mm
